File: usb.sch (KiCad schematic (older format))
At the start: 6 parts, among them J2101 USB-C/16p, U2101 CH340C

Commit message: übergabe an 3ahel
Parts:
- J2101: footprint rs232-sniffer:USB_C_Receptacle_LCSC_C167321 -> htl_connectors:USB_C_Receptacle_LCSC_C167321; Notes USB-C, 16-polig -> USB-C, 16-polig, USB 2.0
Connections:
- net D+: now reaches J2101.A6 (D+), J2101.B6 (D+), U2101.5 (UD+)
- net D-: now reaches J2101.A7 (D-), J2101.B7 (D-), U2101.6 (UD-)
Changed lines of the file:
@@
 Sheet 25 27
 Title "RS-232 Sniffer"
-Date "2020-10-07"
+Date "2020-10-09"
 Rev "v20.0.0-dev"
 Comp "HTL-Steyr"
-Comment1 "Karl Zeilhofer"
+Comment1 "Prof. Karl Zeilhofer"
 Comment2 ""
 Comment3 ""
@@
 AR Path="/5F8070C3/5F7FB5B8/5F70A555" Ref="#PWR?"  Part="1"
 AR Path="/5F8AD0E2/5F7FB5B8/5F70A555" Ref="#PWR02502"  Part="1"
-F 0 "#PWR02502" H 1650 3950 50  0001 C CNN
+AR Path="/5FA85ABF/5F7FB5B8/5F70A555" Ref="#PWR02509"  Part="1"
+F 0 "#PWR02509" H 1650 3950 50  0001 C CNN
 F 1 "GND" H 1655 4027 50  0000 C CNN
 F 2 "" H 1650 4200 50  0001 C CNN
@@
 AR Path="/5F8070C3/5F7FB5B8/5F711352" Ref="#PWR?"  Part="1"
 AR Path="/5F8AD0E2/5F7FB5B8/5F711352" Ref="#PWR02506"  Part="1"
-F 0 "#PWR02506" H 3800 3900 50  0001 C CNN
+AR Path="/5FA85ABF/5F7FB5B8/5F711352" Ref="#PWR02513"  Part="1"
+F 0 "#PWR02513" H 3800 3900 50  0001 C CNN
 F 1 "GND" H 3805 3977 50  0000 C CNN
 F 2 "" H 3800 4150 50  0001 C CNN
@@
 AR Path="/5F8070C3/5F7FB5B8/5F711A46" Ref="C?"  Part="1"
 AR Path="/5F8AD0E2/5F7FB5B8/5F711A46" Ref="C2503"  Part="1"
-F 0 "C2503" V 3848 2400 50  0000 C CNN
+AR Path="/5FA85ABF/5F7FB5B8/5F711A46" Ref="C2506"  Part="1"
+F 0 "C2506" V 3848 2400 50  0000 C CNN
 F 1 "100n" V 3939 2400 50  0000 C CNN
 F 2 "Capacitor_SMD:C_0603_1608Metric" H 4138 2250 50  0001 C CNN
@@
 AR Path="/5F8070C3/5F7FB5B8/5F7120DC" Ref="#PWR?"  Part="1"
 AR Path="/5F8AD0E2/5F7FB5B8/5F7120DC" Ref="#PWR02507"  Part="1"
-F 0 "#PWR02507" H 4350 2150 50  0001 C CNN
+AR Path="/5FA85ABF/5F7FB5B8/5F7120DC" Ref="#PWR02514"  Part="1"
+F 0 "#PWR02514" H 4350 2150 50  0001 C CNN
 F 1 "GND" V 4355 2272 50  0000 R CNN
 F 2 "" H 4350 2400 50  0001 C CNN
@@
 AR Path="/5F8070C3/5F7FB5B8/5F715116" Ref="U?"  Part="1"
 AR Path="/5F8AD0E2/5F7FB5B8/5F715116" Ref="U2501"  Part="1"
-F 0 "U2501" H 3400 3900 50  0000 C CNN
+AR Path="/5FA85ABF/5F7FB5B8/5F715116" Ref="U2502"  Part="1"
+F 0 "U2502" H 3400 3900 50  0000 C CNN
 F 1 "CH340C" H 4000 2750 50  0000 C CNN
 F 2 "Package_SO:SOIC-16_3.9x9.9mm_P1.27mm" H 3850 2750 50  0001 L CNN
@@
 AR Path="/5F8070C3/5F7FB5B8/5F764796" Ref="R?"  Part="1"
 AR Path="/5F8AD0E2/5F7FB5B8/5F764796" Ref="R2501"  Part="1"
-F 0 "R2501" V 2993 3000 50  0000 C CNN
+AR Path="/5FA85ABF/5F7FB5B8/5F764796" Ref="R2502"  Part="1"
+F 0 "R2502" V 2993 3000 50  0000 C CNN
 F 1 "100R" V 3084 3000 50  0000 C CNN
 F 2 "Resistor_SMD:R_0603_1608Metric" V 3130 3000 50  0001 C CNN
@@
 AR Path="/5F8070C3/5F7FB5B8/5F764C96" Ref="#PWR?"  Part="1"
 AR Path="/5F8AD0E2/5F7FB5B8/5F764C96" Ref="#PWR02503"  Part="1"
-F 0 "#PWR02503" H 2900 2750 50  0001 C CNN
+AR Path="/5FA85ABF/5F7FB5B8/5F764C96" Ref="#PWR02510"  Part="1"
+F 0 "#PWR02510" H 2900 2750 50  0001 C CNN
 F 1 "GND" H 2905 2827 50  0000 C CNN
 F 2 "" H 2900 3000 50  0001 C CNN
@@
 AR Path="/5F8070C3/5F7FB5B8/5F7675CD" Ref="C?"  Part="1"
 AR Path="/5F8AD0E2/5F7FB5B8/5F7675CD" Ref="C2502"  Part="1"
-F 0 "C2502" V 3148 2400 50  0000 C CNN
+AR Path="/5FA85ABF/5F7FB5B8/5F7675CD" Ref="C2505"  Part="1"
+F 0 "C2505" V 3148 2400 50  0000 C CNN
 F 1 "100n" V 3239 2400 50  0000 C CNN
 F 2 "Capacitor_SMD:C_0603_1608Metric" H 3438 2250 50  0001 C CNN
@@
 AR Path="/5F8070C3/5F7FB5B8/5F767C48" Ref="#PWR?"  Part="1"
 AR Path="/5F8AD0E2/5F7FB5B8/5F767C48" Ref="#PWR02504"  Part="1"
-F 0 "#PWR02504" H 3150 2150 50  0001 C CNN
+AR Path="/5FA85ABF/5F7FB5B8/5F767C48" Ref="#PWR02511"  Part="1"
+F 0 "#PWR02511" H 3150 2150 50  0001 C CNN
 F 1 "GND" V 3155 2272 50  0000 R CNN
 F 2 "" H 3150 2400 50  0001 C CNN
@@
 AR Path="/5F8070C3/5F7FB5B8/5F6E6B4D" Ref="J?"  Part="1"
 AR Path="/5F8AD0E2/5F7FB5B8/5F6E6B4D" Ref="J2501"  Part="1"
-F 0 "J2501" H 1757 4067 50  0000 C CNN
+AR Path="/5FA85ABF/5F7FB5B8/5F6E6B4D" Ref="J2502"  Part="1"
+F 0 "J2502" H 1757 4067 50  0000 C CNN
 F 1 "USB-C/16p" H 1757 3976 50  0000 C CNN
-F 2 "rs232-sniffer:USB_C_Receptacle_LCSC_C167321" H 1800 3200 50  0001 C CNN
+F 2 "htl_connectors:USB_C_Receptacle_LCSC_C167321" H 1800 3200 50  0001 C CNN
 F 3 "https://www.usb.org/sites/default/files/documents/usb_type-c.zip" H 1800 3200 50  0001 C CNN
 F 4 "Jing Extension" H 1650 3200 50  0001 C CNN "Manufacturer"
@@
 F 9 "100" H 1650 3200 50  0001 C CNN "PriceForQty"
 F 10 "https://lcsc.com/product-detail/USB-Connectors_Jing-Extension-of-the-Electronic-Co-C167321_C167321.html" H 1650 3200 50  0001 C CNN "Weblink"
-F 11 "USB-C, 16-polig" H 1650 3200 50  0001 C CNN "Notes"
+F 11 "USB-C, 16-polig, USB 2.0" H 1650 3200 50  0001 C CNN "Notes"
 F 12 "C167321" H 1650 3200 50  0001 C CNN "DistOrderNr"
 F 13 "C167321" H 1650 3200 50  0001 C CNN "ManPartNr"
@@
 AR Path="/5F7F8851/5F7FB5B8/5F96D29B" Ref="#PWR02105"  Part="1"
 AR Path="/5F8AD0E2/5F7FB5B8/5F96D29B" Ref="#PWR02505"  Part="1"
-F 0 "#PWR02505" H 3800 1550 50  0001 C CNN
+AR Path="/5FA85ABF/5F7FB5B8/5F96D29B" Ref="#PWR02512"  Part="1"
+F 0 "#PWR02512" H 3800 1550 50  0001 C CNN
 F 1 "+3V3" H 3815 1873 50  0000 C CNN
 F 2 "" H 3800 1700 50  0001 C CNN
@@
 AR Path="/5F7F8851/5F7FB5B8/5F81810D" Ref="#FLG02101"  Part="1"
 AR Path="/5F8AD0E2/5F7FB5B8/5F81810D" Ref="#FLG02501"  Part="1"
-F 0 "#FLG02501" H 2250 2375 50  0001 C CNN
+AR Path="/5FA85ABF/5F7FB5B8/5F81810D" Ref="#FLG02502"  Part="1"
+F 0 "#FLG02502" H 2250 2375 50  0001 C CNN
 F 1 "PWR_FLAG" V 2250 2428 50  0000 L CNN
 F 2 "" H 2250 2300 50  0001 C CNN
@@
 AR Path="/5F8070C3/5F7FB5B8/5F818ECB" Ref="#PWR?"  Part="1"
 AR Path="/5F8AD0E2/5F7FB5B8/5F818ECB" Ref="#PWR02501"  Part="1"
-F 0 "#PWR02501" H 1350 4350 50  0001 C CNN
+AR Path="/5FA85ABF/5F7FB5B8/5F818ECB" Ref="#PWR02508"  Part="1"
+F 0 "#PWR02508" H 1350 4350 50  0001 C CNN
 F 1 "GND" H 1355 4427 50  0000 C CNN
 F 2 "" H 1350 4600 50  0001 C CNN
@@
 AR Path="/5F8070C3/5F7FB5B8/5F819C70" Ref="C?"  Part="1"
 AR Path="/5F8AD0E2/5F7FB5B8/5F819C70" Ref="C2501"  Part="1"
-F 0 "C2501" H 1465 4304 50  0000 L CNN
+AR Path="/5FA85ABF/5F7FB5B8/5F819C70" Ref="C2504"  Part="1"
+F 0 "C2504" H 1465 4304 50  0000 L CNN
 F 1 "100n" H 1465 4395 50  0000 L CNN
 F 2 "Capacitor_SMD:C_0603_1608Metric" H 1388 4200 50  0001 C CNN
@@
 Wire Wire Line
 	1350 4500 1350 4600
+Text Label 2700 3200 0    50   ~ 0
+D+
+Text Label 2700 3300 0    50   ~ 0
+D-
 $EndSCHEMATC
