File: rs232-sniffer.sch (KiCad schematic (older format))
At the start: 30 parts, among them J1 Stiftleiste 2x8, J2 DB9_Female, J3 DB9_Male, J4 DB9_Female, J5 DB9_Female

Commit message: version marius wasinger
Parts:
- J2: footprint Connector_Dsub:DSUB-9_Female_EdgeMount_P2.77mm -> rs232-sniffer:DSUB-9_Female_EdgeMount_P2.77mm
- J3: footprint Connector_Dsub:DSUB-9_Male_EdgeMount_P2.77mm -> rs232-sniffer:DSUB-9_Male_EdgeMount_P2.77mm
- J4, J5: footprint Connector_Dsub:DSUB-9_Female_Vertical_P2.77x2.84mm_MountingHoles -> rs232-sniffer:DSUB-9_Female_Vertical_P2.77x2.84mm_MountingHoles
- R1, R10, R2, R20, R3, R30, R4, R40, R6, R60, R7, R70, R8, R80, R9, R90: symbol zeilhofer:R_sig -> rs232-sniffer-rescue:R_sig-zeilhofer
- TP1, TP2, TP3, TP4, TP5, TP6, TP7, TP8, TP9: footprint rs232-sniffer:TestPoint_Pad_5.0x3.0mm -> rs232-sniffer:TestPoint_Pad_5.0x3.0mm_paste
Changed lines of the file:
@@
 F 0 "J2" H 2818 3142 50  0000 C CNN
 F 1 "DB9_Female" H 2818 3051 50  0000 C CNN
-F 2 "Connector_Dsub:DSUB-9_Female_EdgeMount_P2.77mm" H 2900 2450 50  0001 C CNN
+F 2 "rs232-sniffer:DSUB-9_Female_EdgeMount_P2.77mm" H 2900 2450 50  0001 C CNN
 F 3 " ~" H 2900 2450 50  0001 C CNN
 	1    2900 2450
@@
 F 0 "J3" H 9618 1758 50  0000 C CNN
 F 1 "DB9_Male" H 9618 1849 50  0000 C CNN
-F 2 "Connector_Dsub:DSUB-9_Male_EdgeMount_P2.77mm" H 9700 2450 50  0001 C CNN
+F 2 "rs232-sniffer:DSUB-9_Male_EdgeMount_P2.77mm" H 9700 2450 50  0001 C CNN
 F 3 " ~" H 9700 2450 50  0001 C CNN
 	1    9700 2450
@@
 Zum Gerät
 $Comp
-L zeilhofer:R_sig R3
+L rs232-sniffer-rescue:R_sig-zeilhofer R3
 U 1 1 5DE6718C
 P 3600 2450
@@
 $EndComp
 $Comp
-L zeilhofer:R_sig R7
+L rs232-sniffer-rescue:R_sig-zeilhofer R7
 U 1 1 5DE68A5A
 P 3600 2350
@@
 $EndComp
 $Comp
-L zeilhofer:R_sig R4
+L rs232-sniffer-rescue:R_sig-zeilhofer R4
 U 1 1 5DE68CBB
 P 3600 2650
@@
 	3750 2650 4950 2650
 $Comp
-L zeilhofer:R_sig R2
+L rs232-sniffer-rescue:R_sig-zeilhofer R2
 U 1 1 5DE68E79
 P 8850 2250
@@
 	3750 2350 4750 2350
 $Comp
-L zeilhofer:R_sig R8
+L rs232-sniffer-rescue:R_sig-zeilhofer R8
 U 1 1 5DE69E8D
 P 8850 2550
@@
 	9000 2550 9400 2550
 $Comp
-L zeilhofer:R_sig R6
+L rs232-sniffer-rescue:R_sig-zeilhofer R6
 U 1 1 5DE6A196
 P 8850 2150
@@
 	9000 2150 9400 2150
 $Comp
-L zeilhofer:R_sig R1
+L rs232-sniffer-rescue:R_sig-zeilhofer R1
 U 1 1 5DE6A435
 P 8850 2050
@@
 	9000 2050 9400 2050
 $Comp
-L zeilhofer:R_sig R9
+L rs232-sniffer-rescue:R_sig-zeilhofer R9
 U 1 1 5DE6A621
 P 8850 2750
@@
 	4650 6000 4500 6000
 $Comp
-L zeilhofer:R_sig R70
+L rs232-sniffer-rescue:R_sig-zeilhofer R70
 U 1 1 5DE6DF29
 P 4750 4650
@@
 F 0 "J4" H 4118 6292 50  0000 C CNN
 F 1 "DB9_Female" H 4118 6201 50  0000 C CNN
-F 2 "Connector_Dsub:DSUB-9_Female_Vertical_P2.77x2.84mm_MountingHoles" H 4200 5600 50  0001 C CNN
+F 2 "rs232-sniffer:DSUB-9_Female_Vertical_P2.77x2.84mm_MountingHoles" H 4200 5600 50  0001 C CNN
 F 3 " ~" H 4200 5600 50  0001 C CNN
 	1    4200 5600
@@
 F 0 "J5" H 6418 6342 50  0000 C CNN
 F 1 "DB9_Female" H 6418 6251 50  0000 C CNN
-F 2 "Connector_Dsub:DSUB-9_Female_Vertical_P2.77x2.84mm_MountingHoles" H 6500 5650 50  0001 C CNN
+F 2 "rs232-sniffer:DSUB-9_Female_Vertical_P2.77x2.84mm_MountingHoles" H 6500 5650 50  0001 C CNN
 F 3 " ~" H 6500 5650 50  0001 C CNN
 	1    6500 5650
@@
 	7050 2150 8700 2150
 $Comp
-L zeilhofer:R_sig R60
+L rs232-sniffer-rescue:R_sig-zeilhofer R60
 U 1 1 5DE86646
 P 7050 5000
@@
 	7350 2750 8700 2750
 $Comp
-L zeilhofer:R_sig R20
+L rs232-sniffer-rescue:R_sig-zeilhofer R20
 U 1 1 5DE88D53
 P 7150 5000
@@
 $EndComp
 $Comp
-L zeilhofer:R_sig R80
+L rs232-sniffer-rescue:R_sig-zeilhofer R80
 U 1 1 5DE8913B
 P 7250 5000
@@
 $EndComp
 $Comp
-L zeilhofer:R_sig R90
+L rs232-sniffer-rescue:R_sig-zeilhofer R90
 U 1 1 5DE892AF
 P 7350 5000
@@
 	4850 2450 5550 2450
 $Comp
-L zeilhofer:R_sig R30
+L rs232-sniffer-rescue:R_sig-zeilhofer R30
 U 1 1 5DE8CAD8
 P 4850 4650
@@
 $EndComp
 $Comp
-L zeilhofer:R_sig R40
+L rs232-sniffer-rescue:R_sig-zeilhofer R40
 U 1 1 5DE8CC3E
 P 4950 4650
@@
 Connection ~ 3400 2850
 $Comp
-L zeilhofer:R_sig R10
+L rs232-sniffer-rescue:R_sig-zeilhofer R10
 U 1 1 5DE86192
 P 6950 5000
@@
 F 0 "TP7" H 4306 4248 50  0000 R CNN
 F 1 "SMD Testpoint" H 4306 4203 50  0001 R CNN
-F 2 "rs232-sniffer:TestPoint_Pad_5.0x3.0mm" H 4550 4200 50  0001 C CNN
+F 2 "rs232-sniffer:TestPoint_Pad_5.0x3.0mm_paste" H 4550 4200 50  0001 C CNN
 F 3 "~" H 4550 4200 50  0001 C CNN
 	1    4350 4200
@@
 F 0 "TP3" H 4306 4348 50  0000 R CNN
 F 1 "SMD Testpoint" H 4306 4303 50  0001 R CNN
-F 2 "rs232-sniffer:TestPoint_Pad_5.0x3.0mm" H 4550 4300 50  0001 C CNN
+F 2 "rs232-sniffer:TestPoint_Pad_5.0x3.0mm_paste" H 4550 4300 50  0001 C CNN
 F 3 "~" H 4550 4300 50  0001 C CNN
 	1    4350 4300
@@
 F 0 "TP4" H 4306 4448 50  0000 R CNN
 F 1 "SMD Testpoint" H 4306 4403 50  0001 R CNN
-F 2 "rs232-sniffer:TestPoint_Pad_5.0x3.0mm" H 4550 4400 50  0001 C CNN
+F 2 "rs232-sniffer:TestPoint_Pad_5.0x3.0mm_paste" H 4550 4400 50  0001 C CNN
 F 3 "~" H 4550 4400 50  0001 C CNN
 	1    4350 4400
@@
 F 0 "TP5" H 4156 2998 50  0000 R CNN
 F 1 "SMD Testpoint" H 4156 2953 50  0001 R CNN
-F 2 "rs232-sniffer:TestPoint_Pad_5.0x3.0mm" H 4400 2950 50  0001 C CNN
+F 2 "rs232-sniffer:TestPoint_Pad_5.0x3.0mm_paste" H 4400 2950 50  0001 C CNN
 F 3 "~" H 4400 2950 50  0001 C CNN
 	1    4200 2950
@@
 F 0 "TP1" H 6556 3098 50  0000 R CNN
 F 1 "SMD Testpoint" H 6556 3053 50  0001 R CNN
-F 2 "rs232-sniffer:TestPoint_Pad_5.0x3.0mm" H 6800 3050 50  0001 C CNN
+F 2 "rs232-sniffer:TestPoint_Pad_5.0x3.0mm_paste" H 6800 3050 50  0001 C CNN
 F 3 "~" H 6800 3050 50  0001 C CNN
 	1    6600 3050
@@
 F 0 "TP6" H 6556 3548 50  0000 R CNN
 F 1 "SMD Testpoint" H 6556 3503 50  0001 R CNN
-F 2 "rs232-sniffer:TestPoint_Pad_5.0x3.0mm" H 6800 3500 50  0001 C CNN
+F 2 "rs232-sniffer:TestPoint_Pad_5.0x3.0mm_paste" H 6800 3500 50  0001 C CNN
 F 3 "~" H 6800 3500 50  0001 C CNN
 	1    6600 3500
@@
 F 0 "TP2" H 6556 3998 50  0000 R CNN
 F 1 "SMD Testpoint" H 6556 3953 50  0001 R CNN
-F 2 "rs232-sniffer:TestPoint_Pad_5.0x3.0mm" H 6800 3950 50  0001 C CNN
+F 2 "rs232-sniffer:TestPoint_Pad_5.0x3.0mm_paste" H 6800 3950 50  0001 C CNN
 F 3 "~" H 6800 3950 50  0001 C CNN
 	1    6600 3950
@@
 F 0 "TP8" H 6556 4448 50  0000 R CNN
 F 1 "SMD Testpoint" H 6556 4403 50  0001 R CNN
-F 2 "rs232-sniffer:TestPoint_Pad_5.0x3.0mm" H 6800 4400 50  0001 C CNN
+F 2 "rs232-sniffer:TestPoint_Pad_5.0x3.0mm_paste" H 6800 4400 50  0001 C CNN
 F 3 "~" H 6800 4400 50  0001 C CNN
 	1    6600 4400
@@
 F 0 "TP9" H 6556 4848 50  0000 R CNN
 F 1 "SMD Testpoint" H 6556 4803 50  0001 R CNN
-F 2 "rs232-sniffer:TestPoint_Pad_5.0x3.0mm" H 6800 4800 50  0001 C CNN
+F 2 "rs232-sniffer:TestPoint_Pad_5.0x3.0mm_paste" H 6800 4800 50  0001 C CNN
 F 3 "~" H 6800 4800 50  0001 C CNN
 	1    6600 4800

Commit message: wip
Parts:
- removed J4, J5: DB9_Female, rs232-sniffer:DSUB-9_Female_Vertical_P2.77x2.84mm_MountingHoles, symbol Connector:DB9_Female
- removed TP1, TP2, TP3, TP4, TP6, TP7, TP8, TP9: SMD Testpoint, rs232-sniffer:TestPoint_Pad_5.0x3.0mm_paste, symbol Connector:TestPoint_Flag
- added C101, C102: 10u/16V, Capacitor_SMD:C_0603_1608Metric, symbol Device:C
- added D101, D102: red/green, rs232-sniffer:LED_LiteOn_LTST-C195KGJRKT, symbol Device:LED_Dual_AACC
- added H101, H102, H103, H104: MountingHole, MountingHole:MountingHole_4mm, symbol Mechanical:MountingHole
- added J104: Stiftleiste 2x9, rs232-sniffer:PinHeader_2x09_P2.54mm_Vertical_SMD, symbol Connector_Generic:Conn_02x09_Odd_Even
- added R104: 4k7, Resistor_SMD:R_0603_1608Metric, symbol htl_passives:R_sig
- added R108, R109, R110, R111, R112, R121, R122, R123: 100R, Resistor_SMD:R_0603_1608Metric, symbol htl_passives:R_sig
- added R113: 1k, Resistor_SMD:R_0603_1608Metric, symbol htl_passives:R_sig
- added R118, R120: 0R, Resistor_SMD:R_0603_1608Metric, symbol Device:R
- added SW101: DIP-Switch 8, Button_Switch_SMD:SW_DIP_SPSTx08_Slide_6.7x21.88mm_W8.61mm_P2.54mm_LowProfile, symbol Switch:SW_DIP_x08
- added TP102, TP103: SMD Testpoint, rs232-sniffer:Keystone_5016, symbol Connector:TestPoint_Flag
- added U101: AMS1117-3.3, Package_TO_SOT_SMD:SOT-223-3_TabPin2, symbol Regulator_Linear:AMS1117-3.3
- J101: renamed from J2; footprint rs232-sniffer:DSUB-9_Female_EdgeMount_P2.77mm -> rs232-sniffer:DSUB-9_Female_Vertical_P2.77x2.84mm_MountingHoles; symbol Connector:DB9_Female -> Connector:DB9_Female_MountingHoles; DistOrderNr (none) -> C75748; Distributor (none) -> LCSC; ManPartNr (none) -> DS1033-09FUNSiSS-CT; Manufacturer (none) -> CONNFLY Elec; Notes (none) -> RS232 weiblich; PriceEUR (none) -> 0.063911; PriceForQty (none) -> 150; Weblink (none) -> https://lcsc.com/product-detail/D-Sub-Connectors_D-SUB-9pin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
- J102: renamed from J1; value Stiftleiste 2x8 -> Stiftleiste 2x9; footprint rs232-sniffer:PinHeader_2x08_P2.54mm_Vertical_SMD -> rs232-sniffer:PinHeader_2x09_P2.54mm_Vertical_SMD; symbol Connector_Generic:Conn_02x08_Counter_Clockwise -> Connector_Generic:Conn_02x09_Odd_Even; DistOrderNr (none) -> C88175; Distributor (none) -> LCSC; ManPartNr (none) -> C88175; Manufacturer (none) -> BOOMELE(Boom Precision Elec); Notes (none) -> SMD; PriceEUR (none) -> 0.036; PriceForQty (none) -> 100; Weblink (none) -> https://lcsc.com/product-detail/Pin-Header-Female-Header_BO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
- J103: renamed from J3; footprint rs232-sniffer:DSUB-9_Male_EdgeMount_P2.77mm -> rs232-sniffer:DSUB-9_Male_EdgeMount_P2.77mm_MountingHoles; symbol Connector:DB9_Male -> Connector:DB9_Male_MountingHoles; DistOrderNr (none) -> C75746; Distributor (none) -> LCSC; ManPartNr (none) -> DS1033-09MUNSiSS; Manufacturer (none) -> CONNFLY Elec; Notes (none) -> RS232 männlich; PriceEUR (none) -> 0.059745; PriceForQty (none) -> 150; Weblink (none) -> https://lcsc.com/product-detail/D-Sub-Connectors_D-SUB-9pin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
- R101: renamed from R7; value 0R -> 100R; footprint Resistor_SMD:R_1206_3216Metric_Pad1.42x1.75mm_HandSolder -> Resistor_SMD:R_0603_1608Metric; symbol rs232-sniffer-rescue:R_sig-zeilhofer -> htl_passives:R_sig; DistOrderNr (none) -> C25201; Distributor (none) -> LCSC; ManPartNr (none) -> 0603WAJ0101T5E; Manufacturer (none) -> UNI-ROYAL; Notes (none) -> 100R, 5%, 100mW; PriceEUR (none) -> 0.000563; PriceForQty (none) -> 1000; Weblink (none) -> https://lcsc.com/product-detail/Chip-Resistor-Surface-Mount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
- R102: renamed from R3; value 0R -> 100R; footprint Resistor_SMD:R_1206_3216Metric_Pad1.42x1.75mm_HandSolder -> Resistor_SMD:R_0603_1608Metric; symbol rs232-sniffer-rescue:R_sig-zeilhofer -> htl_passives:R_sig; DistOrderNr (none) -> C25201; Distributor (none) -> LCSC; ManPartNr (none) -> 0603WAJ0101T5E; Manufacturer (none) -> UNI-ROYAL; Notes (none) -> 100R, 5%, 100mW; PriceEUR (none) -> 0.000563; PriceForQty (none) -> 1000; Weblink (none) -> https://lcsc.com/product-detail/Chip-Resistor-Surface-Mount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
- R103: renamed from R4; value 0R -> 100R; footprint Resistor_SMD:R_1206_3216Metric_Pad1.42x1.75mm_HandSolder -> Resistor_SMD:R_0603_1608Metric; symbol rs232-sniffer-rescue:R_sig-zeilhofer -> htl_passives:R_sig; DistOrderNr (none) -> C25201; Distributor (none) -> LCSC; ManPartNr (none) -> 0603WAJ0101T5E; Manufacturer (none) -> UNI-ROYAL; Notes (none) -> 100R, 5%, 100mW; PriceEUR (none) -> 0.000563; PriceForQty (none) -> 1000; Weblink (none) -> https://lcsc.com/product-detail/Chip-Resistor-Surface-Mount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
- R105: renamed from R70; value 0R -> 100R; footprint Resistor_SMD:R_1206_3216Metric_Pad1.42x1.75mm_HandSolder -> Resistor_SMD:R_0603_1608Metric; symbol rs232-sniffer-rescue:R_sig-zeilhofer -> htl_passives:R_sig; DistOrderNr (none) -> C25201; Distributor (none) -> LCSC; ManPartNr (none) -> 0603WAJ0101T5E; Manufacturer (none) -> UNI-ROYAL; Notes (none) -> 100R, 5%, 100mW; PriceEUR (none) -> 0.000563; PriceForQty (none) -> 1000; Weblink (none) -> https://lcsc.com/product-detail/Chip-Resistor-Surface-Mount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
- R106: renamed from R30; value 0R -> 100R; footprint Resistor_SMD:R_1206_3216Metric_Pad1.42x1.75mm_HandSolder -> Resistor_SMD:R_0603_1608Metric; symbol rs232-sniffer-rescue:R_sig-zeilhofer -> htl_passives:R_sig; DistOrderNr (none) -> C25201; Distributor (none) -> LCSC; ManPartNr (none) -> 0603WAJ0101T5E; Manufacturer (none) -> UNI-ROYAL; Notes (none) -> 100R, 5%, 100mW; PriceEUR (none) -> 0.000563; PriceForQty (none) -> 1000; Weblink (none) -> https://lcsc.com/product-detail/Chip-Resistor-Surface-Mount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
- R107: renamed from R40; value 0R -> 100R; footprint Resistor_SMD:R_1206_3216Metric_Pad1.42x1.75mm_HandSolder -> Resistor_SMD:R_0603_1608Metric; symbol rs232-sniffer-rescue:R_sig-zeilhofer -> htl_passives:R_sig; DistOrderNr (none) -> C25201; Distributor (none) -> LCSC; ManPartNr (none) -> 0603WAJ0101T5E; Manufacturer (none) -> UNI-ROYAL; Notes (none) -> 100R, 5%, 100mW; PriceEUR (none) -> 0.000563; PriceForQty (none) -> 1000; Weblink (none) -> https://lcsc.com/product-detail/Chip-Resistor-Surface-Mount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
- R114: renamed from R10; value 0R -> 100R; footprint Resistor_SMD:R_1206_3216Metric_Pad1.42x1.75mm_HandSolder -> Resistor_SMD:R_0603_1608Metric; symbol rs232-sniffer-rescue:R_sig-zeilhofer -> htl_passives:R_sig; DistOrderNr (none) -> C25201; Distributor (none) -> LCSC; ManPartNr (none) -> 0603WAJ0101T5E; Manufacturer (none) -> UNI-ROYAL; Notes (none) -> 100R, 5%, 100mW; PriceEUR (none) -> 0.000563; PriceForQty (none) -> 1000; Weblink (none) -> https://lcsc.com/product-detail/Chip-Resistor-Surface-Mount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
- R115: renamed from R60; value 0R -> 100R; footprint Resistor_SMD:R_1206_3216Metric_Pad1.42x1.75mm_HandSolder -> Resistor_SMD:R_0603_1608Metric; symbol rs232-sniffer-rescue:R_sig-zeilhofer -> htl_passives:R_sig; DistOrderNr (none) -> C25201; Distributor (none) -> LCSC; ManPartNr (none) -> 0603WAJ0101T5E; Manufacturer (none) -> UNI-ROYAL; Notes (none) -> 100R, 5%, 100mW; PriceEUR (none) -> 0.000563; PriceForQty (none) -> 1000; Weblink (none) -> https://lcsc.com/product-detail/Chip-Resistor-Surface-Mount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
- R116: renamed from R20; value 0R -> 100R; footprint Resistor_SMD:R_1206_3216Metric_Pad1.42x1.75mm_HandSolder -> Resistor_SMD:R_0603_1608Metric; symbol rs232-sniffer-rescue:R_sig-zeilhofer -> htl_passives:R_sig; DistOrderNr (none) -> C25201; Distributor (none) -> LCSC; ManPartNr (none) -> 0603WAJ0101T5E; Manufacturer (none) -> UNI-ROYAL; Notes (none) -> 100R, 5%, 100mW; PriceEUR (none) -> 0.000563; PriceForQty (none) -> 1000; Weblink (none) -> https://lcsc.com/product-detail/Chip-Resistor-Surface-Mount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
- R117: renamed from R80; value 0R -> 100R; footprint Resistor_SMD:R_1206_3216Metric_Pad1.42x1.75mm_HandSolder -> Resistor_SMD:R_0603_1608Metric; symbol rs232-sniffer-rescue:R_sig-zeilhofer -> htl_passives:R_sig; DistOrderNr (none) -> C25201; Distributor (none) -> LCSC; ManPartNr (none) -> 0603WAJ0101T5E; Manufacturer (none) -> UNI-ROYAL; Notes (none) -> 100R, 5%, 100mW; PriceEUR (none) -> 0.000563; PriceForQty (none) -> 1000; Weblink (none) -> https://lcsc.com/product-detail/Chip-Resistor-Surface-Mount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
- R119: renamed from R90; value 0R -> 100R; footprint Resistor_SMD:R_1206_3216Metric_Pad1.42x1.75mm_HandSolder -> Resistor_SMD:R_0603_1608Metric; symbol rs232-sniffer-rescue:R_sig-zeilhofer -> htl_passives:R_sig; DistOrderNr (none) -> C25201; Distributor (none) -> LCSC; ManPartNr (none) -> 0603WAJ0101T5E; Manufacturer (none) -> UNI-ROYAL; Notes (none) -> 100R, 5%, 100mW; PriceEUR (none) -> 0.000563; PriceForQty (none) -> 1000; Weblink (none) -> https://lcsc.com/product-detail/Chip-Resistor-Surface-Mount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
- R124: renamed from R1; value 0R -> 100R; footprint Resistor_SMD:R_1206_3216Metric_Pad1.42x1.75mm_HandSolder -> Resistor_SMD:R_0603_1608Metric; symbol rs232-sniffer-rescue:R_sig-zeilhofer -> htl_passives:R_sig; DistOrderNr (none) -> C25201; Distributor (none) -> LCSC; ManPartNr (none) -> 0603WAJ0101T5E; Manufacturer (none) -> UNI-ROYAL; Notes (none) -> 100R, 5%, 100mW; PriceEUR (none) -> 0.000563; PriceForQty (none) -> 1000; Weblink (none) -> https://lcsc.com/product-detail/Chip-Resistor-Surface-Mount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
- R125: renamed from R6; value 0R -> 100R; footprint Resistor_SMD:R_1206_3216Metric_Pad1.42x1.75mm_HandSolder -> Resistor_SMD:R_0603_1608Metric; symbol rs232-sniffer-rescue:R_sig-zeilhofer -> htl_passives:R_sig; DistOrderNr (none) -> C25201; Distributor (none) -> LCSC; ManPartNr (none) -> 0603WAJ0101T5E; Manufacturer (none) -> UNI-ROYAL; Notes (none) -> 100R, 5%, 100mW; PriceEUR (none) -> 0.000563; PriceForQty (none) -> 1000; Weblink (none) -> https://lcsc.com/product-detail/Chip-Resistor-Surface-Mount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
- R126: renamed from R2; value 0R -> 100R; footprint Resistor_SMD:R_1206_3216Metric_Pad1.42x1.75mm_HandSolder -> Resistor_SMD:R_0603_1608Metric; symbol rs232-sniffer-rescue:R_sig-zeilhofer -> htl_passives:R_sig; DistOrderNr (none) -> C25201; Distributor (none) -> LCSC; ManPartNr (none) -> 0603WAJ0101T5E; Manufacturer (none) -> UNI-ROYAL; Notes (none) -> 100R, 5%, 100mW; PriceEUR (none) -> 0.000563; PriceForQty (none) -> 1000; Weblink (none) -> https://lcsc.com/product-detail/Chip-Resistor-Surface-Mount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
- R127: renamed from R8; value 0R -> 100R; footprint Resistor_SMD:R_1206_3216Metric_Pad1.42x1.75mm_HandSolder -> Resistor_SMD:R_0603_1608Metric; symbol rs232-sniffer-rescue:R_sig-zeilhofer -> htl_passives:R_sig; DistOrderNr (none) -> C25201; Distributor (none) -> LCSC; ManPartNr (none) -> 0603WAJ0101T5E; Manufacturer (none) -> UNI-ROYAL; Notes (none) -> 100R, 5%, 100mW; PriceEUR (none) -> 0.000563; PriceForQty (none) -> 1000; Weblink (none) -> https://lcsc.com/product-detail/Chip-Resistor-Surface-Mount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
- R128: renamed from R9; value 0R -> 100R; footprint Resistor_SMD:R_1206_3216Metric_Pad1.42x1.75mm_HandSolder -> Resistor_SMD:R_0603_1608Metric; symbol rs232-sniffer-rescue:R_sig-zeilhofer -> htl_passives:R_sig; DistOrderNr (none) -> C25201; Distributor (none) -> LCSC; ManPartNr (none) -> 0603WAJ0101T5E; Manufacturer (none) -> UNI-ROYAL; Notes (none) -> 100R, 5%, 100mW; PriceEUR (none) -> 0.000563; PriceForQty (none) -> 1000; Weblink (none) -> https://lcsc.com/product-detail/Chip-Resistor-Surface-Mount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
- TP101: renamed from TP5; footprint rs232-sniffer:TestPoint_Pad_5.0x3.0mm_paste -> rs232-sniffer:Keystone_5016; DistOrderNr (none) -> C238129; Distributor (none) -> LCSC; ManPartNr (none) -> 5016; Manufacturer (none) -> Keystone; Notes (none) -> SMD Testöse; PriceEUR (none) -> 0.084; PriceForQty (none) -> 1000; Weblink (none) -> https://lcsc.com/product-detail/Test-Points-Test-Rings_Keys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
Connections:
- net GND: now also C101.2, C102.2, D101.3 (K1), D102.3 (K1), J104.10 (Pin_10), J104.12 (Pin_12), J104.14 (Pin_14), J104.16 (Pin_16), J104.18 (Pin_18), J104.2 (Pin_2), J104.4 (Pin_4), J104.6 (Pin_6), J104.8 (Pin_8), J104.9 (Pin_9), TP102.1, TP103.1, U101.1 (GND)
- net LEDs A/Signal1: now reaches J101.1, J102.1 (Pin_1)
- net LEDs A/Signal1: now also SW101.13
- net LEDs A/Signal2: now reaches J101.2
- net LEDs A/Signal2: now also J102.5 (Pin_5), SW101.15; no longer J102.3 (Pin_3)
- net LEDs A/Signal6: now reaches J101.6
- net LEDs A/Signal6: now also J102.3 (Pin_3), SW101.14; no longer J102.2 (Pin_2)
- net LEDs A/Signal8: now reaches J101.8
- net LEDs A/Signal8: now also J102.11 (Pin_11), SW101.16; no longer J102.6 (Pin_6)
- net LEDs A/Signal9: now reaches J101.9
- net LEDs A/Signal9: now also J102.15 (Pin_15); no longer J102.8 (Pin_8)
- net LEDs B/Signal3: now reaches J103.3
- net LEDs B/Signal3: now also J102.10 (Pin_10), SW101.11; no longer J102.12 (Pin_12)
- net LEDs B/Signal4: now reaches J103.4
- net LEDs B/Signal4: now also J102.14 (Pin_14), SW101.10; no longer J102.10 (Pin_10)
- net LEDs A/Signal4: now reaches J102.13 (Pin_13)
- net LEDs A/Signal4: now also R103.2, R107.1, R108.1; no longer J103.7
- net UART Hub L/~CTS: now reaches R105.2
- net UART Hub L/~DCD: now reaches R107.2
- net UART Hub L/RxD: now reaches R106.2
- net UART Hub R/~DCD: now reaches R114.2
- net UART Hub R/RxD: now reaches R116.2
- net UART Hub R/~DSR: now reaches R115.2
- net UART Hub R/~CTS: now reaches R117.2
- net ClearToSend renamed LEDs B/Signal8
- net LEDs B/Signal8: now also J102.12 (Pin_12); no longer J102.11 (Pin_11)
- net DataCarrierDetect renamed LEDs B/Signal1
- net LEDs B/Signal1: now also J102.2 (Pin_2); no longer J102.16 (Pin_16)
- net DataSetReady renamed LEDs B/Signal6
- net LEDs B/Signal6: now also J102.4 (Pin_4); no longer J102.15 (Pin_15)
- removed net DataTerminalReady: J102.7 (Pin_7), R103.2, R107.1
- net ReadyToReceive renamed LEDs A/Signal7
- net LEDs A/Signal7: now also J102.7 (Pin_7); no longer J102.4 (Pin_4)
- net ReceiveData renamed LEDs B/Signal2
- net LEDs B/Signal2: now also J102.6 (Pin_6); no longer J102.14 (Pin_14)
- net RingIndicator renamed LEDs B/Signal9
- net LEDs B/Signal9: now also J102.16 (Pin_16); no longer J102.9 (Pin_9)
- net Sig3 renamed LEDs A/Signal3
- net LEDs A/Signal3: now also J102.9 (Pin_9); no longer J102.5 (Pin_5)
- new net: R111.2, SW101.3
- new net: R110.2, SW101.2
- new net: R109.2, SW101.1
- new net: R123.2, SW101.8
- new net: R122.2, SW101.7
- new net: R121.2, SW101.6
- new net: R112.2, SW101.4
- new net: D101.1 (A1), R104.2
- new net: D102.1 (A1), R113.2
- new net +3V3: C102.1, J104.11 (Pin_11), J104.13 (Pin_13), J104.15 (Pin_15), J104.17 (Pin_17), R113.1, U101.2 (VO)
- new net +5V: C101.1, J104.1 (Pin_1), J104.3 (Pin_3), J104.5 (Pin_5), J104.7 (Pin_7), R104.1, R118.2, R120.2, U101.3 (VI)
- new net LEDs B/Signal7: J102.8 (Pin_8), J103.7, SW101.9
- new net Shield: J101.0 (PAD), J103.0 (PAD)
- new net UART Hub L/TxD: R110.1
- new net UART Hub L/USB-Power: R118.1
- new net UART Hub L/~DSR: R108.2
- new net UART Hub L/~DTR: R111.1, R112.1
- new net UART Hub L/~RTR: R109.1
- new net UART Hub R/TxD: R121.1
- new net UART Hub R/USB-Power: R120.1
- new net UART Hub R/~DTR: R122.1
- new net UART Hub R/~RTR: R123.1
- no-connect marks 7 -> 9
Other:
- note added: "(1) RTR hatte früher (vor 1980) RTS (Request to send geheißen)"
- note added: "ClearToSend"
- note added: "DataCarrierDetect"
- note added: "DataSetReady"
- note added: "DataTerminalReady"
- note added: "Direkte \nVerdrahtung"
- note added: "ReadyToReceive (1)"
- note added: "ReceiveData"
- note added: "RingIndicator"
- note added: "TransmitData"
- note added: "Verdrahtung\nwie Nullmodem"
- note added: "Vom PC (DTE)"
- note added: "Zum Gerät\n(DCE)"
- note added: "hoher Strom wg. \nmöglicher 5V Eingangspegel\nund folglich Strom über \nSchutzdiode im CH340C in die 3V3 Versorgung"
- note added: "siehe Wikipedia"
- note removed: "Bemerkung zu Pin 7: \nFrüher (ca. vor 1990) war die \nBedeutung "Request to Send" \nmit gleicher Richtung."
- note removed: "Gerät zum\nZum Sniff-PC"
- note removed: "PC zum\nZum Sniff-PC"
- note removed: "Vom PC"
- note removed: "Zum Gerät"
- moved on the sheet: R101, R102, R103, R105, R106, R107, R114, R115, R116, R117, R119, TP101

Commit message: übergabe an 3ahel
Parts:
- removed R101, R102, R103, R124, R125, R126, R127, R128: 100R, Resistor_SMD:R_0603_1608Metric, symbol htl_passives:R_sig
- added Item101, Item102, Item103, Item104, Item105, Item106, Item107, Item108: Jumper, ~, symbol htl_virtual:Item
- C101, C102: value 10u/16V -> 10u/16V/X5R; footprint Capacitor_SMD:C_0603_1608Metric -> Capacitor_SMD:C_0805_2012Metric; DistOrderNr (none) -> C1713; Distributor (none) -> LCSC; ManPartNr (none) -> CL21A106KOQNNNE; Manufacturer (none) -> Samsung; Notes (none) -> 10uF ±10% 16V X5R; PriceEUR (none) -> 0.011386; PriceForQty (none) -> 200; Weblink (none) -> https://lcsc.com/product-detail/Multilayer-Ceramic-Capacito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
- D101, D102: footprint rs232-sniffer:LED_LiteOn_LTST-C195KGJRKT -> htl_smd:LED_LiteOn_LTST-C195KGJRKT
- J101: footprint rs232-sniffer:DSUB-9_Female_Vertical_P2.77x2.84mm_MountingHoles -> htl_connectors:DSUB-9_Female_EdgeMount_P2.77mm; symbol Connector:DB9_Female_MountingHoles -> htl_connectors:RS232_DB9_Female
- J102, J104: footprint rs232-sniffer:PinHeader_2x09_P2.54mm_Vertical_SMD -> Connector_PinHeader_2.54mm:PinHeader_2x09_P2.54mm_Vertical_SMD
- J103: footprint rs232-sniffer:DSUB-9_Male_EdgeMount_P2.77mm_MountingHoles -> htl_connectors:DSUB-9_Male_EdgeMount_P2.77mm; symbol Connector:DB9_Male_MountingHoles -> htl_connectors:RS232_DB9_Male
- R120: renamed from R113; DistOrderNr C103662 -> C103209; ManPartNr RTT03472JTP -> RTT03102JTP; Notes 4.7kΩ ±5% 0.1W ±100ppm/℃ -> 1kΩ ±5% 0.1W ±100ppm/℃; PriceEUR 0.000527 -> 0.000556; Weblink https://lcsc.com/product-detail/Chip-Resistor-Surface-Mount_RALEC-RTT03472JTP_C103662.html -> https://lcsc.com/product-detail/Chip-Resistor-Surface-Mount_1KR-102-5_C103209.html
- TP101, TP102, TP103: footprint rs232-sniffer:Keystone_5016 -> htl_smd:Keystone_5016
- renumbered R105 to R101, R106 to R102, R107 to R103, R108 to R104, R109 to R105, R110 to R106, R111 to R107, R112 to R108, R121 to R109, R122 to R110, R123 to R111, R114 to R112, R115 to R113, R116 to R114, R117 to R115, R119 to R116, R120 to R117, R104 to R119
Connections:
- net GND: now also J102.17 (Pin_17), J102.18 (Pin_18)
- net LEDs A/Signal1: now also J102.9 (Pin_9), SW101.15; no longer J102.1 (Pin_1), SW101.13
- net LEDs A/Signal2: now also J102.7 (Pin_7), SW101.16; no longer J102.5 (Pin_5), SW101.15
- net LEDs A/Signal3: now also J101.3 (TxD), J102.1 (Pin_1), R101.1; no longer J102.9 (Pin_9), R102.1
- net LEDs A/Signal4: now also J101.4 (DTR), J102.3 (Pin_3), R102.1; no longer J102.13 (Pin_13), R104.1
- net LEDs A/Signal6: now also J102.11 (Pin_11); no longer J102.3 (Pin_3)
- net LEDs A/Signal7: now also J101.7 (RTR(RTS)), J102.5 (Pin_5), R104.1; no longer J102.7 (Pin_7), R101.1
- net LEDs A/Signal8: now also J102.13 (Pin_13), SW101.13; no longer J102.11 (Pin_11), SW101.16
- net LEDs B/Signal1: now also J102.10 (Pin_10), J103.1 (DCD), R113.1; no longer J102.2 (Pin_2), R112.1
- net LEDs B/Signal2: now also J102.8 (Pin_8), J103.2 (RxD), R112.1; no longer J102.6 (Pin_6), R114.1
- net LEDs B/Signal3: now also J102.2 (Pin_2); no longer J102.10 (Pin_10)
- net LEDs B/Signal4: now also J102.4 (Pin_4); no longer J102.14 (Pin_14)
- net LEDs B/Signal6: now also J102.12 (Pin_12), J103.6 (DSR), R114.1; no longer J102.4 (Pin_4), R113.1
- net LEDs B/Signal7: now also J102.6 (Pin_6); no longer J102.8 (Pin_8)
- net LEDs B/Signal8: now also J102.14 (Pin_14), J103.8 (CTS); no longer J102.12 (Pin_12)
- net LEDs B/Signal9: now also J103.9 (RI)
- net UART Hub L/RxD: now also R101.2; no longer R102.2
- net UART Hub L/TxD: now also R105.1; no longer R106.1
- net UART Hub L/~CTS: now also R104.2; no longer R101.2
- net UART Hub L/~DCD: now also R102.2; no longer R103.2
- net UART Hub L/~DSR: now also R103.2; no longer R104.2
- net UART Hub L/~DTR: now also R106.1; no longer R108.1
- net UART Hub L/~RTR: now also R108.1; no longer R105.1
- net UART Hub R/RxD: now also R112.2; no longer R114.2
- net UART Hub R/~DCD: now also R113.2; no longer R112.2
- net UART Hub R/~DSR: now also R114.2; no longer R113.2
- net LEDs A/Signal9: no longer names the net of J101.9 (RI), J102.15 (Pin_15)
- removed net Shield: J101.0 (PAD), J103.0 (PAD)
- no-connect marks 9 -> 7
Other:
- note added: "gn"
- note added: "hoher Strom wg. \nmöglicher 5V Eingangspegel\nund folglich Strom über \nSchutzdiode im CH340C in die 3V3 Versorgung\nWird über LED abgeleitet."
- note added: "rt"
- note removed: "hoher Strom wg. \nmöglicher 5V Eingangspegel\nund folglich Strom über \nSchutzdiode im CH340C in die 3V3 Versorgung"
- moved on the sheet: D101, D102, H101, H102, H103, H104, R109, R110, R111, R118, R119, R120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
