File: kicad/rs232-sniffer.kicad_pcb (KiCad board)
At the start: 2 copper layers, 103 x 90 mm, 161 parts, among them J101 DB9_Female, J102 Stiftleiste 2x9, J103 DB9_Male, J104 Stiftleiste 2x9, J2001 Stiftleiste 2x9, J2002 Stiftleiste 2x9, J2401 Stiftleiste 2x9, J2402 Buchsenleiste 1x6, horizontal, J2403 Stiftleiste 2x9, J2405 Buchsenleiste 1x6, horizontal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

Commit message: fertig geroutet
Parts:
- J2402, J2405: footprint Connector_PinSocket_2.54mm:PinSocket_1x07_P2.54mm_Horizontal -> Connector_PinSocket_2.54mm:PinSocket_1x06_P2.54mm_Horizontal
- moved R117 32.7 mm to (109.5, 119.5)
- moved J2002 21.0 mm to (131.0, 84.0)
- moved J2403 21.0 mm to (40.0, 84.0)
- moved J2402 19.8 mm to (125.5, 97.8)
- moved J2405 17.6 mm to (45.8, 110.5)
- moved R118 13.0 mm to (65.2, 121.5)
- moved R2401 4.81 mm to (121.5, 108.2)
- moved R2402 4.81 mm to (121.5, 109.8)
- moved R2403 4.81 mm to (121.5, 105.2)
- moved R2404 4.81 mm to (121.5, 106.8)
- moved R2405 4.81 mm to (121.5, 111.2)
- moved R2406 4.81 mm to (121.5, 103.8)
- moved R2407 4.81 mm to (121.5, 112.8)
- moved R2408 4.81 mm to (121.5, 114.2)
Routing:
- net +5V: track 141.1 -> 176.9 mm, vias 5 -> 4
- net /UART Hub R/USB-Power: track 45.3 -> 11.3 mm
- net Net-(J2001-Pad3): track 47.9 -> 18.7 mm, vias 0 -> 1
- net /UART Hub L/UART - RS232 1/UART_Rx2: track 0.00 -> 28.9 mm
- net Net-(J2001-Pad7): track 38.5 -> 13.1 mm, vias 2 -> 0
- net Net-(J2001-Pad5): track 41.9 -> 17.5 mm, vias 2 -> 1
- net /UART Hub R/UART - RS232 1/UART_Rx1: track 7.74 -> 31.0 mm, vias 0 -> 2
- net /UART Hub L/~DCD: track 0.00 -> 22.9 mm, vias 0 -> 2
- net Net-(J2403-Pad1): track 37.1 -> 15.1 mm, vias 2 -> 0
- net Net-(J2403-Pad10): track 33.5 -> 11.8 mm, vias 2 -> 0
- net /UART Hub L/UART - RS232 2/UART_Rx1: track 6.12 -> 27.7 mm, vias 2 -> 3
- net Net-(J2403-Pad5): track 35.4 -> 13.8 mm, vias 2 -> 0
- net Net-(J2403-Pad3): track 35.9 -> 14.7 mm
- net Net-(J2403-Pad11): track 32.6 -> 11.4 mm
- net Net-(J2403-Pad7): track 33.6 -> 12.8 mm
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- added copper zone on F.Cu, net +3V3
Other:
- board text added: "RS-232 Sniffer HTL Steyr"

Commit message: V20.0.0 fertig zur Leiterplattenbestellung, BOM export, PDF, Gerber
Parts:
- moved R109 1.84 mm to (89.1, 81.8)
- moved R110 1.84 mm to (90.8, 81.8)
- moved R111 1.84 mm to (92.6, 81.8)
- moved R105 1.80 mm to (76.5, 81.8)
- moved R106 1.80 mm to (78.2, 81.8)
- moved R107 1.80 mm to (80.0, 81.8)
- moved R108 1.80 mm to (81.8, 81.8)
- moved C2506 0.25 mm to (54.0, 114.0)
- moved R118 0.15 mm to (65.2, 121.3)
Routing:
- net +3V3: track 205.4 -> 201.2 mm
- net Net-(R107-Pad2): track 4.19 -> 7.06 mm
- net Net-(R108-Pad2): track 4.52 -> 7.18 mm
- net Net-(R111-Pad2): track 4.07 -> 6.59 mm
- net /UART Hub L/~DTR: track 32.2 -> 30.4 mm
- net /UART Hub L/TxD: track 25.2 -> 23.4 mm
- net Net-(R106-Pad2): track 3.95 -> 5.75 mm
- net Net-(R105-Pad2): track 4.28 -> 6.08 mm
- net /UART Hub L/USB - UART/TxD: track 22.6 -> 24.3 mm
- net /UART Hub L/USB - UART/~RI: track 31.7 -> 33.3 mm
- net Net-(R109-Pad2): track 4.40 -> 6.03 mm
- net Net-(R110-Pad2): track 4.07 -> 5.67 mm
- net /UART Hub L/~DCD: track 22.9 -> 21.5 mm
- net /LEDs A/Signal6: track 100.8 -> 99.5 mm
- net /UART Hub R/TxD: track 23.6 -> 22.6 mm
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Other:
- rule solder_mask_min_width: 0.25 -> 0.1
- board text added: "+"
- board text added: "0/3.3V"
- board text added: "1:1"
- board text added: "3.3V UART"
- board text added: "3V3"
- board text added: "5V"
- board text added: "CTS"
- board text added: "D+"
- board text added: "D-"
- board text added: "DCD"
- board text added: "DSR"
- board text added: "DTR"
- board text added: "GND"
- board text added: "Null- Modem"
- board text added: "RI"
- board text added: "RS-232 Sniffer, HTL Steyr"
- board text added: "RS232"
- board text added: "RTR"
- board text added: "RxD"
- board text added: "TxD"
- board text added: "UART"
- board text added: "USB"
- board text added: "USB-C USB 2.0"
- board text added: "closed"
- board text added: "open"
- board text added: "±3...15V"
- board text removed: "RS-232 Sniffer HTL Steyr"
