File: kicad/rs232-sniffer.kicad_pcb (KiCad board)
At the start: 2 copper layers, 103 x 90 mm, 161 parts, among them J101 DB9_Female, J102 Stiftleiste 2x9, J103 DB9_Male, J104 Stiftleiste 2x9, J2001 Stiftleiste 2x9, J2002 Stiftleiste 2x9, J2401 Stiftleiste 2x9, J2402 Buchsenleiste 1x6, horizontal, J2403 Stiftleiste 2x9, J2405 Buchsenleiste 1x6, horizontal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

Commit message: v20.0.1 fertig, 30 Stk bestellt
Parts:
- turned D1001 to 90 degrees
- turned D1201 to 90 degrees
- turned D1301 to 90 degrees
- turned D1401 to 90 degrees
- turned D1501 to 90 degrees
- turned D1601 to 90 degrees
- turned D1701 to 90 degrees
- turned D1801 to 90 degrees
- turned D1901 to 90 degrees
- turned D301 to 90 degrees
- turned D401 to 90 degrees
- turned D501 to 90 degrees
- turned D601 to 90 degrees
- turned D701 to 90 degrees
- turned D801 to 90 degrees
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Routing:
- net /LEDs A/Signal6: track 99.5 -> 76.2 mm
- net Net-(D701-Pad1): track 13.6 -> 4.94 mm
- net /LEDs B/Signal9: track 72.9 -> 80.5 mm
- net /LEDs B/Signal8: track 73.0 -> 80.2 mm
- net /LEDs B/Signal1: track 71.6 -> 77.3 mm
- net /LEDs B/Signal6: track 72.8 -> 78.5 mm
- net /LEDs B/Signal2: track 70.8 -> 76.3 mm
- net /LEDs B/Signal7: track 65.4 -> 70.3 mm
- net /LEDs B/Signal4: track 65.6 -> 69.8 mm
- net /LEDs B/Signal3: track 68.7 -> 70.6 mm
- net /LEDs A/Signal4: track 72.0 -> 70.1 mm
- net Net-(D801-Pad1): track 3.40 -> 4.94 mm
- net Net-(D601-Pad1): track 3.40 -> 4.94 mm
- net Net-(D501-Pad1): track 3.40 -> 4.94 mm
- net Net-(D401-Pad1): track 3.40 -> 4.94 mm
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Other:
- board text added: "LED GN = HIGH LED RT = LOW"
- board text added: "V20.0.1"
- board text removed: "V20.0.0"
