File: kicad/uart-hub.sch (KiCad schematic (older format))
At the start: 20 parts, among them J2001 Stiftleiste 2x9, J2002 Buchsenleiste 1x6, horizontal, J2002 Stiftleiste 2x9, SW2001 DIP-Switch 8

Commit message: fertig geroutet
Parts:
- J2002: footprint Connector_PinSocket_2.54mm:PinSocket_1x07_P2.54mm_Horizontal -> Connector_PinSocket_2.54mm:PinSocket_1x06_P2.54mm_Horizontal

Commit message: V20.0.0 fertig zur Leiterplattenbestellung, BOM export, PDF, Gerber
Changed lines of the file:
@@
 Sheet 20 27
 Title "RS-232 Sniffer"
-Date "2020-10-09"
-Rev "v20.0.0-dev"
+Date "2020-11-13"
+Rev "v20.0.0"
 Comp "HTL-Steyr"
 Comment1 "Prof. Karl Zeilhofer"
@@
 	6200 4150 6200 3650
 Connection ~ 6200 3650
+Wire Notes Line
+	2350 4400 4800 4400
 $EndSCHEMATC

Commit message: BOM vervollständigt
Parts:
- J2002: DistOrderNr (none) -> C225514; Distributor (none) -> LCSC; ManPartNr (none) -> A2541HWR-6P; Manufacturer (none) -> CJT(Changjiang Connectors); Notes (none) -> Buchsenleiste, 1x6, 2.54mm, gewinkelt; PriceEUR (none) -> 0.13; PriceForQty (none) -> 30; Weblink (none) -> https://www.lcsc.com/product-detail/Female-Headers_CJT-Chan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
Changed lines of the file:
@@
 F 2 "Connector_PinSocket_2.54mm:PinSocket_1x06_P2.54mm_Horizontal" H 3750 5650 50  0001 C CNN
 F 3 "" H 3750 5650 50  0001 C CNN
+F 4 "C225514" H 3750 5650 50  0001 C CNN "DistOrderNr"
+F 5 "LCSC" H 3750 5650 50  0001 C CNN "Distributor"
+F 6 "A2541HWR-6P" H 3750 5650 50  0001 C CNN "ManPartNr"
+F 7 "CJT(Changjiang Connectors)" H 3750 5650 50  0001 C CNN "Manufacturer"
+F 8 "Buchsenleiste, 1x6, 2.54mm, gewinkelt" H 3750 5650 50  0001 C CNN "Notes"
+F 9 "0.13" H 3750 5650 50  0001 C CNN "PriceEUR"
+F 10 "30" H 3750 5650 50  0001 C CNN "PriceForQty"
+F 11 "https://www.lcsc.com/product-detail/Female-Headers_CJT-Changjiang-Connectors-A2541HWR-6P_C225514.html" H 3750 5650 50  0001 C CNN "Weblink"
 	1    3750 5650
 	0    1    1    0
