File: kicad/led.sch (KiCad schematic (older format))
At the start: 3 parts

Commit message: V20.0.0 fertig zur Leiterplattenbestellung, BOM export, PDF, Gerber
Parts:
- D1201: symbol Device:LED_Dual_AACC -> htl_semiconductors:LED_Dual_green-red
Other:
- note removed: "gn"
- note removed: "rt"
Changed lines of the file:
@@
 $Descr A4 11693 8268
 encoding utf-8
-Sheet 3 27
+Sheet 12 27
 Title "RS-232 Sniffer"
-Date "2020-10-09"
-Rev "v20.0.0-dev"
+Date "2020-11-13"
+Rev "v20.0.0"
 Comp "HTL-Steyr"
 Comment1 "Prof. Karl Zeilhofer"
@@
 Wire Wire Line
 	5200 3750 5350 3750
-Text Notes 5800 3650 1    50   ~ 0
-gn
-Text Notes 5800 4150 1    50   ~ 0
-rt
-$Comp
-L Device:LED_Dual_AACC D1201
-U 1 1 5F74784B
-P 5800 3850
-AR Path="/5F87EA32/5F813BE3/5F74784B" Ref="D1201"  Part="1"
-AR Path="/5F80F0BB/5F813BE3/5F74784B" Ref="D301"  Part="1"
-AR Path="/5F80F0BB/5F813C65/5F74784B" Ref="D401"  Part="1"
-AR Path="/5F80F0BB/5F813CCB/5F74784B" Ref="D501"  Part="1"
-AR Path="/5F80F0BB/5F813D49/5F74784B" Ref="D601"  Part="1"
-AR Path="/5F80F0BB/5F813D9D/5F74784B" Ref="D701"  Part="1"
-AR Path="/5F80F0BB/5F813DD9/5F74784B" Ref="D801"  Part="1"
-AR Path="/5F80F0BB/5F813E3D/5F74784B" Ref="D901"  Part="1"
-AR Path="/5F80F0BB/5F813E87/5F74784B" Ref="D1001"  Part="1"
-AR Path="/5F87EA32/5F813C65/5F74784B" Ref="D1301"  Part="1"
-AR Path="/5F87EA32/5F813CCB/5F74784B" Ref="D1401"  Part="1"
-AR Path="/5F87EA32/5F813D49/5F74784B" Ref="D1501"  Part="1"
-AR Path="/5F87EA32/5F813D9D/5F74784B" Ref="D1601"  Part="1"
-AR Path="/5F87EA32/5F813DD9/5F74784B" Ref="D1701"  Part="1"
-AR Path="/5F87EA32/5F813E3D/5F74784B" Ref="D1801"  Part="1"
-AR Path="/5F87EA32/5F813E87/5F74784B" Ref="D1901"  Part="1"
-F 0 "D1901" V 5600 4250 50  0000 L CNN
-F 1 "red/green" H 4700 3700 50  0000 L CNN
-F 2 "htl_smd:LED_LiteOn_LTST-C195KGJRKT" H 5830 3850 50  0001 C CNN
-F 3 "https://datasheet.lcsc.com/szlcsc/1811100910_Lite-On-LTST-C195KGJRKT_C125104.pdf" H 5830 3850 50  0001 C CNN
-F 4 "LiteOn" H 5800 3850 50  0001 C CNN "Manufacturer"
-F 5 "LTST-C195KGJRKT" H 5800 3850 50  0001 C CNN "ManPartNr"
-F 6 "LCSC" H 5800 3850 50  0001 C CNN "Distributor"
-F 7 "C125104" H 5800 3850 50  0001 C CNN "DistOrderNr"
-F 8 "0.023" H 5800 3850 50  0001 C CNN "PriceEUR"
-F 9 "1000" H 5800 3850 50  0001 C CNN "PriceForQty"
-F 10 "https://lcsc.com/product-detail/Light-Emitting-Diodes-LED_Lite-On-LTST-C195KGJRKT_C125104.html" H 5800 3850 50  0001 C CNN "Weblink"
-F 11 "Dual LED" H 5800 3850 50  0001 C CNN "Notes"
-	1    5800 3850
-	-1   0    0    -1
-$EndComp
 Wire Wire Line
 	6550 3750 6750 3750
@@
 AR Path="/5F87EA32/5F813E3D/5DEC45FD" Ref="#PWR01801"  Part="1"
 AR Path="/5F87EA32/5F813E87/5DEC45FD" Ref="#PWR01901"  Part="1"
-F 0 "#PWR01901" H 6750 3500 50  0001 C CNN
+F 0 "#PWR01201" H 6750 3500 50  0001 C CNN
 F 1 "GND" V 6755 3622 50  0000 R CNN
 F 2 "" H 6750 3750 50  0001 C CNN
@@
 AR Path="/5F87EA32/5F813E3D/5DEC44D0" Ref="R1801"  Part="1"
 AR Path="/5F87EA32/5F813E87/5DEC44D0" Ref="R1901"  Part="1"
-F 0 "R1901" V 6193 3750 50  0000 C CNN
+F 0 "R1201" V 6193 3750 50  0000 C CNN
 F 1 "4k7" V 6284 3750 50  0000 C CNN
 F 2 "Resistor_SMD:R_0603_1608Metric" V 6330 3750 50  0001 C CNN
@@
 AR Path="/5F87EA32/5F813E3D/5F74E0AC" Ref="TP1801"  Part="1"
 AR Path="/5F87EA32/5F813E87/5F74E0AC" Ref="TP1901"  Part="1"
-F 0 "TP1901" H 5200 3975 50  0000 C CNN
+F 0 "TP1201" H 5200 3975 50  0000 C CNN
 F 1 "SMD Testpoint" H 5200 3884 50  0000 C CNN
 F 2 "htl_smd:Keystone_5016" H 5400 3650 50  0001 C CNN
@@
 Text Notes 5200 2800 0    63   ~ 0
 Grün: High (-3...-15V)\nRot: Low (+3...+15V)
+$Comp
+L htl_semiconductors:LED_Dual_green-red D1201
+U 1 1 5F74784B
+P 5800 3850
+AR Path="/5F87EA32/5F813BE3/5F74784B" Ref="D1201"  Part="1"
+AR Path="/5F80F0BB/5F813BE3/5F74784B" Ref="D301"  Part="1"
+AR Path="/5F80F0BB/5F813C65/5F74784B" Ref="D401"  Part="1"
+AR Path="/5F80F0BB/5F813CCB/5F74784B" Ref="D501"  Part="1"
+AR Path="/5F80F0BB/5F813D49/5F74784B" Ref="D601"  Part="1"
+AR Path="/5F80F0BB/5F813D9D/5F74784B" Ref="D701"  Part="1"
+AR Path="/5F80F0BB/5F813DD9/5F74784B" Ref="D801"  Part="1"
+AR Path="/5F80F0BB/5F813E3D/5F74784B" Ref="D901"  Part="1"
+AR Path="/5F80F0BB/5F813E87/5F74784B" Ref="D1001"  Part="1"
+AR Path="/5F87EA32/5F813C65/5F74784B" Ref="D1301"  Part="1"
+AR Path="/5F87EA32/5F813CCB/5F74784B" Ref="D1401"  Part="1"
+AR Path="/5F87EA32/5F813D49/5F74784B" Ref="D1501"  Part="1"
+AR Path="/5F87EA32/5F813D9D/5F74784B" Ref="D1601"  Part="1"
+AR Path="/5F87EA32/5F813DD9/5F74784B" Ref="D1701"  Part="1"
+AR Path="/5F87EA32/5F813E3D/5F74784B" Ref="D1801"  Part="1"
+AR Path="/5F87EA32/5F813E87/5F74784B" Ref="D1901"  Part="1"
+F 0 "D1201" V 5600 4250 50  0000 L CNN
+F 1 "red/green" H 4700 3700 50  0000 L CNN
+F 2 "htl_smd:LED_LiteOn_LTST-C195KGJRKT" H 5830 3850 50  0001 C CNN
+F 3 "https://datasheet.lcsc.com/szlcsc/1811100910_Lite-On-LTST-C195KGJRKT_C125104.pdf" H 5830 3850 50  0001 C CNN
+F 4 "LiteOn" H 5800 3850 50  0001 C CNN "Manufacturer"
+F 5 "LTST-C195KGJRKT" H 5800 3850 50  0001 C CNN "ManPartNr"
+F 6 "LCSC" H 5800 3850 50  0001 C CNN "Distributor"
+F 7 "C125104" H 5800 3850 50  0001 C CNN "DistOrderNr"
+F 8 "0.023" H 5800 3850 50  0001 C CNN "PriceEUR"
+F 9 "1000" H 5800 3850 50  0001 C CNN "PriceForQty"
+F 10 "https://lcsc.com/product-detail/Light-Emitting-Diodes-LED_Lite-On-LTST-C195KGJRKT_C125104.html" H 5800 3850 50  0001 C CNN "Weblink"
+F 11 "Dual LED" H 5800 3850 50  0001 C CNN "Notes"
+	1    5800 3850
+	-1   0    0    -1
+$EndComp
 $EndSCHEMATC

Commit message: postcommit
Parts:
- R301: ManPartNr RTT03472JTP -> RTT03472JTP
Changed lines of the file:
@@
 F 4 "C103662" H 6400 3750 50  0001 C CNN "DistOrderNr"
 F 5 "LCSC" H 6400 3750 50  0001 C CNN "Distributor"
-F 6 "RTT03472JTP" H 6400 3750 50  0001 C CNN "ManPartNr"
+F 6 "RTT03472JTP" H 6400 3750 50  0001 C CNN "ManPartNr"
 F 7 "RALEC" H 6400 3750 50  0001 C CNN "Manufacturer"
 F 8 "4.7kΩ ±5% 0.1W ±100ppm/℃" H 6400 3750 50  0001 C CNN "Notes"
