File: kicad/rs232-sniffer.sch (KiCad schematic (older format))
At the start: 45 parts, among them J101 DB9_Female, J102 Stiftleiste 2x9, J103 DB9_Male, J104 Stiftleiste 2x9, SW101 DIP-Switch 8, U101 AMS1117-3.3

Commit message: V20.0.0 fertig zur Leiterplattenbestellung, BOM export, PDF, Gerber
Parts:
- D101, D102: symbol Device:LED_Dual_AACC -> htl_semiconductors:LED_Dual_green-red
Changed lines of the file:
@@
 Sheet 1 27
 Title "RS-232 Sniffer"
-Date "2020-10-09"
-Rev "v20.0.0-dev"
+Date "2020-11-13"
+Rev "v20.0.0"
 Comp "HTL-Steyr"
 Comment1 "Prof. Karl Zeilhofer"
@@
 $EndComp
 $Comp
-L Device:LED_Dual_AACC D?
+L htl_semiconductors:LED_Dual_green-red D?
 U 1 1 5FB4C524
 P 10200 4200
@@
 $EndComp
 $Comp
-L Device:LED_Dual_AACC D?
+L htl_semiconductors:LED_Dual_green-red D?
 U 1 1 5FADBE3A
 P 8700 4200

Commit message: BOM vervollständigt
Parts:
- R117, R118: DistOrderNr (none) -> C101250; ManPartNr (none) -> CR0603JA0000G; Manufacturer (none) -> LIZ Elec; Notes (none) -> 0R Resistor, 1608; Weblink (none) -> https://www.lcsc.com/product-detail/Chip-Resistor-Surface-M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
- R119: ManPartNr RTT03472JTP -> RTT03472JTP
Changed lines of the file:
@@
 F 1 "0R" V 6094 6350 50  0000 C CNN
 F 2 "Resistor_SMD:R_0603_1608Metric" V 6230 6350 50  0001 C CNN
-F 3 "" H 6300 6350 50  0001 C CNN
-F 4 "" H 6300 6350 50  0001 C CNN "DistOrderNr"
+F 3 "https://datasheet.lcsc.com/lcsc/1810170215_LIZ-Elec-CR0603JA0000G_C101250.pdf" H 6300 6350 50  0001 C CNN
+F 4 "C101250" H 6300 6350 50  0001 C CNN "DistOrderNr"
 F 5 "LCSC" H 6300 6350 50  0001 C CNN "Distributor"
-F 6 "" H 6300 6350 50  0001 C CNN "ManPartNr"
-F 7 "" H 6300 6350 50  0001 C CNN "Manufacturer"
-F 8 "" H 6300 6350 50  0001 C CNN "Notes"
+F 6 "CR0603JA0000G" H 6300 6350 50  0001 C CNN "ManPartNr"
+F 7 "LIZ Elec " H 6300 6350 50  0001 C CNN "Manufacturer"
+F 8 "0R Resistor, 1608" H 6300 6350 50  0001 C CNN "Notes"
 F 9 "" H 6300 6350 50  0001 C CNN "PriceEUR"
 F 10 "" H 6300 6350 50  0001 C CNN "PriceForQty"
-F 11 "" H 6300 6350 50  0001 C CNN "Weblink"
+F 11 "https://www.lcsc.com/product-detail/Chip-Resistor-Surface-Mount_LIZ-Elec-CR0603JA0000G_C101250.html" H 6300 6350 50  0001 C CNN "Weblink"
 	1    6300 6350
 	0    -1   -1   0
@@
 F 1 "0R" V 6450 6200 50  0000 C CNN
 F 2 "Resistor_SMD:R_0603_1608Metric" V 6230 6200 50  0001 C CNN
-F 3 "" H 6300 6200 50  0001 C CNN
-F 4 "" H 6300 6200 50  0001 C CNN "DistOrderNr"
+F 3 "https://datasheet.lcsc.com/lcsc/1810170215_LIZ-Elec-CR0603JA0000G_C101250.pdf" H 6300 6200 50  0001 C CNN
+F 4 "C101250" H 6300 6200 50  0001 C CNN "DistOrderNr"
 F 5 "LCSC" H 6300 6200 50  0001 C CNN "Distributor"
-F 6 "" H 6300 6200 50  0001 C CNN "ManPartNr"
-F 7 "" H 6300 6200 50  0001 C CNN "Manufacturer"
-F 8 "" H 6300 6200 50  0001 C CNN "Notes"
+F 6 "CR0603JA0000G" H 6300 6200 50  0001 C CNN "ManPartNr"
+F 7 "LIZ Elec " H 6300 6200 50  0001 C CNN "Manufacturer"
+F 8 "0R Resistor, 1608" H 6300 6200 50  0001 C CNN "Notes"
 F 9 "" H 6300 6200 50  0001 C CNN "PriceEUR"
 F 10 "" H 6300 6200 50  0001 C CNN "PriceForQty"
-F 11 "" H 6300 6200 50  0001 C CNN "Weblink"
+F 11 "https://www.lcsc.com/product-detail/Chip-Resistor-Surface-Mount_LIZ-Elec-CR0603JA0000G_C101250.html" H 6300 6200 50  0001 C CNN "Weblink"
 	1    6300 6200
 	0    -1   -1   0
@@
 F 4 "C103662" H 8200 4300 50  0001 C CNN "DistOrderNr"
 F 5 "LCSC" H 8200 4300 50  0001 C CNN "Distributor"
-F 6 "RTT03472JTP" H 8200 4300 50  0001 C CNN "ManPartNr"
+F 6 "RTT03472JTP" H 8200 4300 50  0001 C CNN "ManPartNr"
 F 7 "RALEC" H 8200 4300 50  0001 C CNN "Manufacturer"
 F 8 "4.7kΩ ±5% 0.1W ±100ppm/℃" H 8200 4300 50  0001 C CNN "Notes"

Commit message: postcommit
Parts:
- R119: ManPartNr RTT03472JTP -> RTT03472JTP
Changed lines of the file:
@@
 F 4 "C103662" H 8200 4300 50  0001 C CNN "DistOrderNr"
 F 5 "LCSC" H 8200 4300 50  0001 C CNN "Distributor"
-F 6 "RTT03472JTP" H 8200 4300 50  0001 C CNN "ManPartNr"
+F 6 "RTT03472JTP" H 8200 4300 50  0001 C CNN "ManPartNr"
 F 7 "RALEC" H 8200 4300 50  0001 C CNN "Manufacturer"
 F 8 "4.7kΩ ±5% 0.1W ±100ppm/℃" H 8200 4300 50  0001 C CNN "Notes"
