File: kicad/uart-rs232.sch (KiCad schematic (older format))
At the start: 6 parts, among them U2201 MAX3232

Commit message: V20.0.0 fertig zur Leiterplattenbestellung, BOM export, PDF, Gerber
Changed lines of the file:
@@
 $Descr A4 11693 8268
 encoding utf-8
-Sheet 26 27
+Sheet 22 27
 Title "RS-232 Sniffer"
-Date "2020-10-09"
-Rev "v20.0.0-dev"
+Date "2020-11-13"
+Rev "v20.0.0"
 Comp "HTL-Steyr"
 Comment1 "Prof. Karl Zeilhofer"
@@
 AR Path="/5FA85ABF/5F7FE442/5F65EF92" Ref="U2602"  Part="1"
 AR Path="/5FA85ABF/5F7FE44C/5F65EF92" Ref="U2702"  Part="1"
-F 0 "U2602" H 4850 4900 50  0000 C CNN
+F 0 "U2601" H 4850 4900 50  0000 C CNN
 F 1 "MAX3232" H 4950 4800 50  0000 C CNN
 F 2 "Package_SO:SOIC-16_3.9x9.9mm_P1.27mm" H 5450 2650 50  0001 L CNN
@@
 AR Path="/5FA85ABF/5F7FE442/5F65EF98" Ref="C2608"  Part="1"
 AR Path="/5FA85ABF/5F7FE44C/5F65EF98" Ref="C2708"  Part="1"
-F 0 "C2608" H 6615 2996 50  0000 L CNN
+F 0 "C2603" H 6615 2996 50  0000 L CNN
 F 1 "100n" H 6615 2905 50  0000 L CNN
 F 2 "Capacitor_SMD:C_0603_1608Metric" H 6538 2800 50  0001 C CNN
@@
 AR Path="/5FA85ABF/5F7FE442/5F65EF9E" Ref="C2606"  Part="1"
 AR Path="/5FA85ABF/5F7FE44C/5F65EF9E" Ref="C2706"  Part="1"
-F 0 "C2606" H 4465 2996 50  0000 L CNN
+F 0 "C2601" H 4465 2996 50  0000 L CNN
 F 1 "100n" H 4465 2905 50  0000 L CNN
 F 2 "Capacitor_SMD:C_0603_1608Metric" H 4388 2800 50  0001 C CNN
@@
 AR Path="/5FA85ABF/5F7FE442/5F65EFA4" Ref="C2610"  Part="1"
 AR Path="/5FA85ABF/5F7FE44C/5F65EFA4" Ref="C2710"  Part="1"
-F 0 "C2610" V 6748 3300 50  0000 C CNN
+F 0 "C2605" V 6748 3300 50  0000 C CNN
 F 1 "100n" V 6839 3300 50  0000 C CNN
 F 2 "Capacitor_SMD:C_0603_1608Metric" H 7038 3150 50  0001 C CNN
@@
 AR Path="/5FA85ABF/5F7FE442/5F65EFAA" Ref="C2609"  Part="1"
 AR Path="/5FA85ABF/5F7FE44C/5F65EFAA" Ref="C2709"  Part="1"
-F 0 "C2609" V 6348 3600 50  0000 C CNN
+F 0 "C2604" V 6348 3600 50  0000 C CNN
 F 1 "100n" V 6439 3600 50  0000 C CNN
 F 2 "Capacitor_SMD:C_0603_1608Metric" H 6638 3450 50  0001 C CNN
@@
 AR Path="/5FA85ABF/5F7FE442/5F65EFB3" Ref="#PWR02610"  Part="1"
 AR Path="/5FA85ABF/5F7FE44C/5F65EFB3" Ref="#PWR02710"  Part="1"
-F 0 "#PWR02710" H 7250 3350 50  0001 C CNN
+F 0 "#PWR02605" H 7250 3350 50  0001 C CNN
 F 1 "GND" V 7255 3472 50  0000 R CNN
 F 2 "" H 7250 3600 50  0001 C CNN
@@
 AR Path="/5FA85ABF/5F7FE442/5F65EFB9" Ref="#PWR02609"  Part="1"
 AR Path="/5FA85ABF/5F7FE44C/5F65EFB9" Ref="#PWR02709"  Part="1"
-F 0 "#PWR02709" H 7250 3050 50  0001 C CNN
+F 0 "#PWR02604" H 7250 3050 50  0001 C CNN
 F 1 "GND" V 7255 3172 50  0000 R CNN
 F 2 "" H 7250 3300 50  0001 C CNN
@@
 AR Path="/5FA85ABF/5F7FE442/5F65EFC4" Ref="C2607"  Part="1"
 AR Path="/5FA85ABF/5F7FE44C/5F65EFC4" Ref="C2707"  Part="1"
-F 0 "C2607" V 5598 2300 50  0000 C CNN
+F 0 "C2602" V 5598 2300 50  0000 C CNN
 F 1 "100n" V 5689 2300 50  0000 C CNN
 F 2 "Capacitor_SMD:C_0603_1608Metric" H 5888 2150 50  0001 C CNN
@@
 AR Path="/5FA85ABF/5F7FE442/5F65EFCC" Ref="#PWR02608"  Part="1"
 AR Path="/5FA85ABF/5F7FE44C/5F65EFCC" Ref="#PWR02708"  Part="1"
-F 0 "#PWR02708" H 6150 2050 50  0001 C CNN
+F 0 "#PWR02603" H 6150 2050 50  0001 C CNN
 F 1 "GND" V 6155 2172 50  0000 R CNN
 F 2 "" H 6150 2300 50  0001 C CNN
@@
 AR Path="/5FA85ABF/5F7FE442/5F65EFD3" Ref="#PWR02607"  Part="1"
 AR Path="/5FA85ABF/5F7FE44C/5F65EFD3" Ref="#PWR02707"  Part="1"
-F 0 "#PWR02707" H 5400 4650 50  0001 C CNN
+F 0 "#PWR02602" H 5400 4650 50  0001 C CNN
 F 1 "GND" H 5405 4727 50  0000 C CNN
 F 2 "" H 5400 4900 50  0001 C CNN
@@
 AR Path="/5FA85ABF/5F7FE442/5F96E1EF" Ref="#PWR02606"  Part="1"
 AR Path="/5FA85ABF/5F7FE44C/5F96E1EF" Ref="#PWR02706"  Part="1"
-F 0 "#PWR02706" H 5400 1950 50  0001 C CNN
+F 0 "#PWR02601" H 5400 1950 50  0001 C CNN
 F 1 "+3V3" H 5415 2273 50  0000 C CNN
 F 2 "" H 5400 2100 50  0001 C CNN

Commit message: postcommit
Parts:
- C2201, C2202, C2203, C2204, C2205: PriceForQty 500 -> 500
Changed lines of the file:
@@
 F 7 "" H 6500 2950 50  0001 C CNN "OrderNr"
 F 8 "0.002141" H 6500 2950 50  0001 C CNN "PriceEUR"
-F 9 "500" H 6500 2950 50  0001 C CNN "PriceForQty"
+F 9 "500" H 6500 2950 50  0001 C CNN "PriceForQty"
 F 10 "https://lcsc.com/product-detail/Multilayer-Ceramic-Capacitors-MLCC-SMD-SMT_Walsin-Tech-Corp-0603B104K160CT_C80516.html" H 6500 2950 50  0001 C CNN "Weblink"
 F 11 "100nF ±10% 16V X7R" H 6500 2950 50  0001 C CNN "Notes"
@@
 F 8 "" H 4350 2950 50  0001 C CNN "PartNr"
 F 9 "0.002141" H 4350 2950 50  0001 C CNN "PriceEUR"
-F 10 "500" H 4350 2950 50  0001 C CNN "PriceForQty"
+F 10 "500" H 4350 2950 50  0001 C CNN "PriceForQty"
 F 11 "https://lcsc.com/product-detail/Multilayer-Ceramic-Capacitors-MLCC-SMD-SMT_Walsin-Tech-Corp-0603B104K160CT_C80516.html" H 4350 2950 50  0001 C CNN "Weblink"
 F 12 "C80516" H 4350 2950 50  0001 C CNN "DistOrderNr"
@@
 F 8 "" H 7000 3300 50  0001 C CNN "PartNr"
 F 9 "0.002141" H 7000 3300 50  0001 C CNN "PriceEUR"
-F 10 "500" H 7000 3300 50  0001 C CNN "PriceForQty"
+F 10 "500" H 7000 3300 50  0001 C CNN "PriceForQty"
 F 11 "https://lcsc.com/product-detail/Multilayer-Ceramic-Capacitors-MLCC-SMD-SMT_Walsin-Tech-Corp-0603B104K160CT_C80516.html" H 7000 3300 50  0001 C CNN "Weblink"
 F 12 "C80516" H 7000 3300 50  0001 C CNN "DistOrderNr"
@@
 F 8 "" H 6600 3600 50  0001 C CNN "PartNr"
 F 9 "0.002141" H 6600 3600 50  0001 C CNN "PriceEUR"
-F 10 "500" H 6600 3600 50  0001 C CNN "PriceForQty"
+F 10 "500" H 6600 3600 50  0001 C CNN "PriceForQty"
 F 11 "https://lcsc.com/product-detail/Multilayer-Ceramic-Capacitors-MLCC-SMD-SMT_Walsin-Tech-Corp-0603B104K160CT_C80516.html" H 6600 3600 50  0001 C CNN "Weblink"
 F 12 "C80516" H 6600 3600 50  0001 C CNN "DistOrderNr"
@@
 F 6 "100nF ±10% 16V X7R" H 5850 2300 50  0001 C CNN "Notes"
 F 7 "0.002141" H 5850 2300 50  0001 C CNN "PriceEUR"
-F 8 "500" H 5850 2300 50  0001 C CNN "PriceForQty"
+F 8 "500" H 5850 2300 50  0001 C CNN "PriceForQty"
 F 9 "https://lcsc.com/product-detail/Multilayer-Ceramic-Capacitors-MLCC-SMD-SMT_Walsin-Tech-Corp-0603B104K160CT_C80516.html" H 5850 2300 50  0001 C CNN "Weblink"
 F 10 "C80516" H 5850 2300 50  0001 C CNN "DistOrderNr"
