File: kicad/usb.sch (KiCad schematic (older format))
At the start: 6 parts, among them J2101 USB-C/16p, U2101 CH340C

Commit message: rework gestartet
Parts:
- J2101: symbol Connector:USB_C_Receptacle_USB2.0 -> rs232-sniffer-rescue:USB_C_Receptacle_USB2.0-Connector
Changed lines of the file:
@@
 	3700 2400 3700 2700
 $Comp
-L Connector:USB_C_Receptacle_USB2.0 J?
+L rs232-sniffer-rescue:USB_C_Receptacle_USB2.0-Connector J?
 U 1 1 5F6E6B4D
 P 1650 3200
@@
 AR Path="/5F8AD0E2/5F7FB5B8/5F6E6B4D" Ref="J2501"  Part="1"
 AR Path="/5FA85ABF/5F7FB5B8/5F6E6B4D" Ref="J2502"  Part="1"
+AR Path="/5F6E6B4D" Ref="J2502"  Part="1"
 F 0 "J2502" H 1757 4067 50  0000 C CNN
 F 1 "USB-C/16p" H 1757 3976 50  0000 C CNN

Commit message: postcommit
Parts:
- C2101, C2102, C2103: PriceForQty 500 -> 500
Changed lines of the file:
@@
 F 8 "" H 4100 2400 50  0001 C CNN "PartNr"
 F 9 "0.002141" H 4100 2400 50  0001 C CNN "PriceEUR"
-F 10 "500" H 4100 2400 50  0001 C CNN "PriceForQty"
+F 10 "500" H 4100 2400 50  0001 C CNN "PriceForQty"
 F 11 "https://lcsc.com/product-detail/Multilayer-Ceramic-Capacitors-MLCC-SMD-SMT_Walsin-Tech-Corp-0603B104K160CT_C80516.html" H 4100 2400 50  0001 C CNN "Weblink"
 F 12 "C80516" H 4100 2400 50  0001 C CNN "DistOrderNr"
@@
 F 8 "" H 3400 2400 50  0001 C CNN "PartNr"
 F 9 "0.002141" H 3400 2400 50  0001 C CNN "PriceEUR"
-F 10 "500" H 3400 2400 50  0001 C CNN "PriceForQty"
+F 10 "500" H 3400 2400 50  0001 C CNN "PriceForQty"
 F 11 "https://lcsc.com/product-detail/Multilayer-Ceramic-Capacitors-MLCC-SMD-SMT_Walsin-Tech-Corp-0603B104K160CT_C80516.html" H 3400 2400 50  0001 C CNN "Weblink"
 F 12 "C80516" H 3400 2400 50  0001 C CNN "DistOrderNr"
@@
 F 8 "" H 1350 4350 50  0001 C CNN "PartNr"
 F 9 "0.002141" H 1350 4350 50  0001 C CNN "PriceEUR"
-F 10 "500" H 1350 4350 50  0001 C CNN "PriceForQty"
+F 10 "500" H 1350 4350 50  0001 C CNN "PriceForQty"
 F 11 "https://lcsc.com/product-detail/Multilayer-Ceramic-Capacitors-MLCC-SMD-SMT_Walsin-Tech-Corp-0603B104K160CT_C80516.html" H 1350 4350 50  0001 C CNN "Weblink"
 F 12 "C80516" H 1350 4350 50  0001 C CNN "DistOrderNr"
